File: MCU Datalogger.kicad_pcb (KiCad board)
At the start: 2 copper layers, 0 parts

Commit message: Setup Pcbnew
Parts:
- added BT1: Battery, Connector_PinHeader_2.54mm:PinHeader_1x02_P2.54mm_Vertical, F.Cu at (236.1, 137.2)
- added C1: 0.1uF, Capacitor_SMD:C_0805_2012Metric, F.Cu at (231.5, 136.4)
- added C2: 0.1uF, Capacitor_SMD:C_0805_2012Metric, F.Cu at (231.5, 139.4)
- added C3: 22pF, Capacitor_SMD:C_0805_2012Metric, F.Cu at (231.5, 142.4)
- added C4: 22pF, Capacitor_SMD:C_0805_2012Metric, F.Cu at (231.5, 145.4)
- added C5: 100nF, Capacitor_SMD:C_0805_2012Metric, F.Cu at (231.5, 148.4)
- added D1: LED, LED_SMD:LED_0805_2012Metric, F.Cu at (236.0, 143.6)
- added D2: LED, LED_SMD:LED_0805_2012Metric, F.Cu at (236.0, 146.6)
- added H1: MountingHole, MountingHole:MountingHole_2.1mm, F.Cu at (211.7, 125.7)
- added H2: MountingHole, MountingHole:MountingHole_2.1mm, F.Cu at (211.7, 131.5)
- added H3: MountingHole, MountingHole:MountingHole_2.1mm, F.Cu at (211.7, 137.2)
- added H4: MountingHole, MountingHole:MountingHole_2.1mm, F.Cu at (211.7, 143.0)
- added J1: Conn_01x04_Pin, Connector_PinHeader_2.54mm:PinHeader_1x04_P2.54mm_Vertical, F.Cu at (247.7, 125.2)
- added J2: Conn_01x09_Pin, Connector_PinHeader_2.54mm:PinHeader_1x09_P2.54mm_Vertical, F.Cu at (243.0, 125.2)
- added J3: Conn_01x04_Pin, Connector_PinHeader_2.54mm:PinHeader_1x04_P2.54mm_Vertical, F.Cu at (252.3, 125.2)
- added J4: Conn_02x03_Odd_Even, Connector_PinHeader_2.54mm:PinHeader_2x03_P2.54mm_Vertical, F.Cu at (247.7, 137.4)
- added R1: 4.7K, Resistor_SMD:R_0805_2012Metric, F.Cu at (216.7, 124.3)
- added R2: 4.7K, Resistor_SMD:R_0805_2012Metric, F.Cu at (216.7, 127.3)
- added R3: 10K, Resistor_SMD:R_0805_2012Metric, F.Cu at (216.7, 130.2)
- added R4: 10K, Resistor_SMD:R_0805_2012Metric, F.Cu at (216.7, 133.2)
- added R5: 10K, Resistor_SMD:R_0805_2012Metric, F.Cu at (216.7, 136.1)
- added R6: 330, Resistor_SMD:R_0805_2012Metric, F.Cu at (216.7, 139.1)
- added R7: 330, Resistor_SMD:R_0805_2012Metric, F.Cu at (216.7, 142.0)
- added U1: 24LC1025, Package_SO:SOIC-8_5.23x5.23mm_P1.27mm, F.Cu at (224.1, 138.3)
- added U2: 24LC1025, Package_SO:SOIC-8_5.23x5.23mm_P1.27mm, F.Cu at (224.1, 145.0)
- added U3: DS1337S+, Footprints:SOIC127P600X175-8N, F.Cu at (234.4, 153.2)
- added U4: ATMEGA328P-AU, Footprints:QFP80P900X900X120-32N, F.Cu at (225.0, 128.9)
- added Y1: 32.768KHz, Crystal:Crystal_SMD_5032-2Pin_5.0x3.2mm_HandSoldering, F.Cu at (224.1, 150.9)
- added Y2: 16MHz, Crystal:Crystal_SMD_5032-2Pin_5.0x3.2mm_HandSoldering, F.Cu at (224.1, 155.7)
